Commit message: map my world

File: src/my_robot/urdf/my_robot.xacro (robot description, xacro)
@@ -8,5 +8,5 @@
     <material>Gazebo/Green</material>
 </gazebo>
-<gazebo reference="camera">
+<gazebo reference="camera_link">
     <material>Gazebo/Blue</material>
 </gazebo>
@@ -37,5 +37,5 @@
   <joint type="fixed" name="camera_joint">
     <origin xyz="0.2 0 0" rpy="0 0 0"/>
-    <child link="camera"/>
+    <child link="camera_link"/>
     <parent link="chassis"/>
     <axis xyz="0 1 0" rpy="0 0 0"/>
@@ -47,4 +47,11 @@
     <axis xyz="0 1 0"/>
   </joint>
+  <joint name="camera_optical_joint" type="fixed">
+    <origin xyz="0 0 0" rpy="-1.5707 0 -1.5707"/>
+    <parent link="camera_link"/>
+    <child link="camera_link_optical"/>
+  </joint>
+  <link name="camera_link_optical">
+  </link>
    <link name='hokuyo'>
 <topicName>/scan</topicName>
@@ -72,5 +79,5 @@
     </visual>
   </link>
-   <link name='camera'>
+   <link name='camera_link'>
 <imageTopicName>rgb/image_raw</imageTopicName>
     <pose>0 0 0 0 0 0</pose>
